File: Kicad/Ax58100-stm32-ethercat/peripherals.kicad_sch (KiCad schematic)
At the start: 56 parts, among them J11 24V Field, J12 DAC, J14 In_opt2, J17 In_opt1, J18 Out_opt, J6 In1-4, J7 In5-8, J8 Output1-2, J9 Output3-4, U4 TLP292-4, U5 TLP292-4, U6 TLP292-4

Commit message: Might be in final shape.
Parts:
- J12: renamed from J11; footprint TerminalBlock:TerminalBlock_bornier-2_P5.08mm -> Connector_Phoenix_MC:PhoenixContact_MCV_1,5_2-G-3.5_1x02_P3.50mm_Vertical
- J13: renamed from J12; footprint TerminalBlock:TerminalBlock_bornier-3_P5.08mm -> Connector_Phoenix_MC:PhoenixContact_MCV_1,5_3-G-3.5_1x03_P3.50mm_Vertical
- J6, J7, J8, J9: footprint TerminalBlock:TerminalBlock_bornier-4_P5.08mm -> Connector_Phoenix_MC:PhoenixContact_MCV_1,5_4-G-3.5_1x04_P3.50mm_Vertical
- R46: value 1k -> 4k7
- renumbered J17 to J14, J14 to J16, R62 to R11, R61 to R14, R60 to R16, R59 to R27, R63 to R30, R64 to R31, R65 to R32, R66 to R33, R67 to R34, R68 to R35, R69 to R36, R70 to R37, U4 to U3, U5 to U4, U6 to U5
Connections:
- net at D3.1 (K), D3.2 (A): now also J7.2 (Pin_2); no longer J7.3 (Pin_3)
- net at D3.1 (K), D3.2 (A): now also J7.3 (Pin_3); no longer J7.2 (Pin_2)
- net at D3.1 (K), D3.2 (A): now also J7.1 (Pin_1); no longer J7.4 (Pin_4)
- net at D3.1 (K), D3.2 (A): now also J7.4 (Pin_4); no longer J7.1 (Pin_1)
- net at D3.1 (K), D3.2 (A): now also J6.4 (Pin_4); no longer J6.1 (Pin_1)
- net at D3.1 (K), D3.2 (A): now also J6.3 (Pin_3); no longer J6.2 (Pin_2)
- net at D3.1 (K), D3.2 (A): now also J6.2 (Pin_2); no longer J6.3 (Pin_3)
- net at D3.1 (K), D3.2 (A): now also J6.1 (Pin_1); no longer J6.4 (Pin_4)

Commit message: Getting ready for fab
Other:
- note added: "Note the reverse order of inputs 1-4 and pins IO12-IO9"
- note added: "Note the reverse order of inputs 1-4 and pins IO8-IO5"
Changed lines of the file:
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@@
+    (effects (font (size 1.27 1.27)) (justify left bottom))
+  )
+  (text "Note the reverse order of \ninputs 1-4 and pins IO12-IO9"
+    (at 122.555 125.73 0)
+    (effects (font (size 1.27 1.27)) (justify left bottom))
+  )
+  (text "Note the reverse order of \ninputs 1-4 and pins IO8-IO5"
+    (at 121.92 52.07 0)
     (effects (font (size 1.27 1.27)) (justify left bottom))
   )
@@
   (symbol (lib_id "Connector_Generic:Conn_01x04") (at 260.985 48.26 0) (unit 1)
     (in_bom yes) (on_board yes) (dnp no)
-    (property "Reference" "J8" (at 260.985 58.7543 0)
+    (property "Reference" "J8" (at 264.795 45.085 0)
       (effects (font (size 1.27 1.27)))
     )
@@
   (symbol (lib_id "Connector_Generic:Conn_01x04") (at 260.985 58.42 0) (unit 1)
     (in_bom yes) (on_board yes) (dnp no)
-    (property "Reference" "J9" (at 260.985 68.9143 0)
-      (effects (font (size 1.27 1.27)))
-    )
+    (property "Reference" "J9" (at 264.795 55.88 0)
+      (effects (font (size 1.27 1.27)))
+    )
